File: ingot-hardware.kicad_sch (KiCad schematic)
At the start: 357 parts, among them J1 USB_C_Receptacle_USB2.0, J2 USB_C_Receptacle_USB2.0, SW1 SW_Diode, SW10 SW_Diode, SW100 SW_Diode, SW101 SW_Diode, SW102 SW_Diode, SW103 SW_Diode, SW104 SW_Diode, SW105 SW_Diode, SW106 SW_Diode, SW107 SW_Diode, SW108 SW_Diode, SW109 SW_Diode, SW11 SW_Diode, SW110 SW_Diode, SW111 SW_Diode, SW112 SW_Diode, SW12 SW_Diode, SW13 SW_Diode, SW14 SW_Diode, SW15 SW_Diode, SW16 SW_Diode, SW17 SW_Diode, SW18 SW_Diode, SW19 SW_Diode, SW2 SW_Diode, SW20 SW_Diode, SW21 SW_Diode, SW22 SW_Diode, SW23 SW_Diode, SW24 SW_Diode, SW25 SW_Diode, SW26 SW_Diode, SW27 SW_Diode, SW28 SW_Diode, SW29 SW_Diode, SW3 SW_Diode, SW30 SW_Diode, SW31 SW_Diode, SW32 SW_Diode, SW33 SW_Diode, SW34 SW_Diode, SW35 SW_Diode, SW36 SW_Diode, SW37 SW_Diode, SW38 SW_Diode, SW39 SW_Diode, SW4 SW_Diode, SW40 SW_Diode, SW41 SW_Diode, SW42 SW_Diode, SW43 SW_Diode, SW44 SW_Diode, SW45 SW_Diode, SW46 SW_Diode, SW47 SW_Diode, SW48 SW_Diode, SW49 SW_Diode, SW5 SW_Diode, SW50 SW_Diode, SW51 SW_Diode, SW52 SW_Diode, SW53 SW_Diode, SW54 SW_Diode, SW55 SW_Diode, SW56 SW_Diode, SW57 SW_Diode, SW58 SW_Diode, SW59 SW_Diode, SW6 SW_Diode, SW60 SW_Diode, SW61 SW_Diode, SW62 SW_Diode, SW63 SW_Diode, SW64 SW_Diode, SW65 SW_Diode, SW66 SW_Diode, SW67 SW_Diode, SW68 SW_Diode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

Commit message: update schematics
Parts:
- Y1, Y2: footprint (none) -> Crystal:Crystal_SMD_HC49-SD_HandSoldering
Changed lines of the file:
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@@
       (effects (font (size 1.27 1.27)) (justify left))
     )
-    (property "Footprint" "" (id 2) (at -57.15 118.11 0)
+    (property "Footprint" "Crystal:Crystal_SMD_HC49-SD_HandSoldering" (id 2) (at -57.15 118.11 0)
       (effects (font (size 1.27 1.27)) hide)
     )
@@
       (effects (font (size 1.27 1.27)) (justify left))
     )
-    (property "Footprint" "" (id 2) (at 355.6 262.89 0)
+    (property "Footprint" "Crystal:Crystal_SMD_HC49-SD_HandSoldering" (id 2) (at 355.6 262.89 0)
       (effects (font (size 1.27 1.27)) hide)
     )
@@
     )
     (path "/e27203e9-3016-4c92-99fd-0eb58bf6200f"
-      (reference "Y1") (unit 1) (value "Crystal") (footprint "")
+      (reference "Y1") (unit 1) (value "Crystal") (footprint "Crystal:Crystal_SMD_HC49-SD_HandSoldering")
     )
     (path "/2c2fadca-3216-4560-8b78-b07e47b0902a"
-      (reference "Y2") (unit 1) (value "Crystal") (footprint "")
+      (reference "Y2") (unit 1) (value "Crystal") (footprint "Crystal:Crystal_SMD_HC49-SD_HandSoldering")
     )
   )
