File: pcb/pcb.kicad_pcb (KiCad board)
At the start: 2 copper layers, 323 x 133 mm, 252 parts, among them SW1 SW_Diode, SW10 SW_Diode, SW100 SW_Diode, SW101 SW_Diode, SW102 SW_Diode, SW103 SW_Diode, SW104 SW_Diode, SW105 SW_Diode, SW106 SW_Diode, SW107 SW_Diode, SW108 SW_Diode, SW11 SW_Diode, SW12 SW_Diode, SW13 SW_Diode, SW14 SW_Diode, SW2 SW_Diode, SW21 SW_Diode, SW22 SW_Diode, SW23 SW_Diode, SW24 SW_Diode, SW25 SW_Diode, SW26 SW_Diode, SW27 SW_Diode, SW28 SW_Diode, SW29 SW_Diode, SW3 SW_Diode, SW30 SW_Diode, SW31 SW_Diode, SW32 SW_Diode, SW33 SW_Diode, SW34 SW_Diode, SW35 SW_Diode, SW36 SW_Diode, SW4 SW_Diode, SW42 SW_Diode, SW43 SW_Diode, SW44 SW_Diode, SW45 SW_Diode, SW46 SW_Diode, SW47 SW_Diode, SW48 SW_Diode, SW49 SW_Diode, SW5 SW_Diode, SW50 SW_Diode, SW51 SW_Diode, SW52 SW_Diode, SW53 SW_Diode, SW54 SW_Diode, SW56 SW_Diode, SW57 SW_Diode, SW6 SW_Diode, SW63 SW_Diode, SW64 SW_Diode, SW65 SW_Diode, SW66 SW_Diode, SW67 SW_Diode, SW68 SW_Diode, SW69 SW_Diode, SW7 SW_Diode, SW70 SW_Diode, SW71 SW_Diode, SW72 SW_Diode, SW73 SW_Diode, SW74 SW_Diode, SW75 SW_Diode, SW76 SW_Diode, SW8 SW_Diode, SW80 SW_Diode, SW81 SW_Diode, SW82 SW_Diode, SW83 SW_Diode, SW84 SW_Diode, SW85 SW_Diode, SW86 SW_Diode, SW87 SW_Diode, SW88 SW_Diode, SW89 SW_Diode, SW9 SW_Diode, SW90 SW_Diode, SW91 SW_Diode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

Commit message: design finished
Parts:
- removed H1: MountingHole, Mounting_Keyboard_Stabilizer:Stabilizer_Cherry_MX_2.00u
- removed H2: MountingHole, Mounting_Keyboard_Stabilizer:Stabilizer_Cherry_MX_6.00u
- D1, D10, D100, D101, D102, D103, D104, D105, D106, D107, D108, D11, D12, D13, D14, D2, D21, D22, D23, D24, D25, D26, D27, D28, D29, D3, D30, D31, D32, D33, D34, D35, D36, D4, D42, D43, D44, D45, D46, D47, D48, D49, D5, D50, D51, D52, D53, D54, D56, D57, D6, D63, D64, D65, D66, D67, D68, D69, D7, D70, D71, D72, D73, D74, D75, D76, D8, D80, D81, D82, D83, D84, D85, D86, D87, D88, D89, D9, D90, D91, D92, D93, D99: footprint Diode_SMD:D_SOD-323 -> easyeda2kicad:SOD-323_L1.8-W1.3-LS2.5-RD
- D113, D114, D115, D116, D117, D118, D119, D120, D121, D122, D123, D124, D125, D126, D128, D129, D130, D131, D132, D133, D134, D135, D136, D137, D138, D139, D140, D141, D142, D143, D144, D145, D146, D147, D148, D149, D150, D151, D152, D153, D154, D155, D156, D157, D158, D159, D160, D161, D162, D163, D164, D165, D166, D167, D168, D169, D170, D171, D172, D173, D174, D175, D176, D177, D178, D182, D183, D186, D187, D188, D212, D213, D214, D215, D216, D217, D218, D219, D220, D221, D222, D223, D224: footprint blackwing:LED-WS2812B-2020 -> easyeda2kicad:LED-SMD_4P-L2.0-W2.0-BR-1
- SW1, SW10, SW100, SW104, SW106, SW107, SW108, SW11, SW12, SW13, SW14, SW2, SW21, SW22, SW23, SW24, SW25, SW26, SW27, SW28, SW29, SW3, SW30, SW31, SW32, SW33, SW35, SW36, SW4, SW43, SW44, SW45, SW46, SW47, SW48, SW49, SW5, SW50, SW51, SW52, SW53, SW54, SW56, SW57, SW6, SW64, SW65, SW66, SW67, SW68, SW69, SW7, SW70, SW71, SW72, SW73, SW74, SW75, SW8, SW81, SW82, SW83, SW84, SW85, SW86, SW87, SW88, SW89, SW9, SW90, SW91, SW93: value SW_Diode -> CPG151101S11-16; footprint blackwing:SW_Cherry_MX_1.00u_PCB -> easyeda2kicad:SMD_KEYBOARD-SW-1.00; moved to B.Cu
- SW101, SW103, SW105, SW80, SW99: value SW_Diode -> CPG151101S11-16; footprint blackwing:SW_Cherry_MX_1.25u_PCB -> easyeda2kicad:SMD_KEYBOARD-SW-1.25; moved to B.Cu
- SW102: value SW_Diode -> CPG151101S11-16; footprint Switch_Keyboard_Cherry_MX:SW_Cherry_MX_PCB_6.00u -> easyeda2kicad:SMD_KEYBOARD-SW-6.00; moved to B.Cu
- SW34: value SW_Diode -> CPG151101S11-16; footprint blackwing:SW_Cherry_MX_2.00u_PCB -> easyeda2kicad:SMD_KEYBOARD-SW-2.00; moved to B.Cu
- SW42: value SW_Diode -> CPG151101S11-16; footprint blackwing:SW_Cherry_MX_1.50u_PCB -> easyeda2kicad:SMD_KEYBOARD-SW-1.50; moved to B.Cu
- SW63, SW92: value SW_Diode -> CPG151101S11-16; footprint blackwing:SW_Cherry_MX_1.75u_PCB -> easyeda2kicad:SMD_KEYBOARD-SW-1.75; moved to B.Cu
- SW76: value SW_Diode -> CPG151101S11-16; footprint Switch_Keyboard_Cherry_MX:SW_Cherry_MX_Plate_ISOEnter -> easyeda2kicad:SMD_KEYBOARD-SW-ENTER-ISO; moved to B.Cu
- moved SW102 3.87 mm to (87.0, 91.5), turned to 180 degrees
- moved SW45 3.44 mm to (39.5, 34.5), turned to 180 degrees
- moved SW46 3.44 mm to (58.5, 34.5), turned to 180 degrees
- moved SW47 3.44 mm to (77.5, 34.5), turned to 180 degrees
- moved SW48 3.44 mm to (96.5, 34.5), turned to 180 degrees
- moved SW49 3.44 mm to (115.5, 34.5), turned to 180 degrees
- moved SW66 3.44 mm to (44.3, 53.5), turned to 180 degrees
- moved SW67 3.44 mm to (63.3, 53.5), turned to 180 degrees
- moved SW68 3.44 mm to (82.3, 53.5), turned to 180 degrees
- moved SW69 3.44 mm to (101.3, 53.5), turned to 180 degrees
- moved SW70 3.44 mm to (120.3, 53.5), turned to 180 degrees
- moved SW25 3.44 mm to (49.0, 15.5), turned to 180 degrees
- moved SW26 3.44 mm to (68.0, 15.5), turned to 180 degrees
- moved SW27 3.44 mm to (87.0, 15.5), turned to 180 degrees
- moved SW28 3.44 mm to (106.0, 15.5), turned to 180 degrees
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Connections:
- D153 pad 1: Net-(D153-SDO) -> Net-(D153-DO)
- D155 pad 1: Net-(D153-SDO) -> Net-(D155-DO)
- D155 pad 3: Net-(D155-SDI) -> Net-(D153-DO)
- D186 pad 3: Net-(D155-SDI) -> Net-(D155-DO)
- D187 pad 2: unconnected-(D187-GND-Pad2) -> GND
- D188 pad 1: SDA -> Net-(D188-DO)
- D188 pad 3: Net-(D188-SDI) -> SDA
- D212 pad 3: Net-(D188-SDI) -> Net-(D188-DO)
- SW102 pad 1: Net-(D102-A) -> C02
- SW102 pad 2: C02 -> Net-(D102-A)
- SW76 pad 1: Net-(D76-A) -> C06
- SW76 pad 2: C06 -> Net-(D76-A)
Routing:
- net Net-(D155-SDI): track 41.0 -> 0.00 mm
- net Net-(D155-DO): track 0.00 -> 41.0 mm
- net Net-(D153-SDO): track 36.1 -> 0.00 mm
- net Net-(D153-DO): track 0.00 -> 36.1 mm
- net C08: track 534.9 -> 564.9 mm, vias 1 -> 2
- net Net-(D188-SDI): track 22.4 -> 0.00 mm
- net Net-(D188-DO): track 0.00 -> 22.4 mm
- net C01: track 398.8 -> 383.1 mm, vias 0 -> 1
- net C07: track 489.9 -> 500.9 mm, vias 0 -> 1
- net Net-(D168-DO): track 29.9 -> 36.0 mm
- net Net-(D113-DI): track 38.7 -> 44.0 mm
- net R09: track 194.5 -> 198.8 mm
- net R06: track 646.2 -> 650.0 mm
- net C02: track 393.7 -> 390.3 mm, vias 0 -> 1
- net R11: track 268.1 -> 271.3 mm
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Other:
- outline, holes or cut-outs redrawn
