File: pcb/pcb.kicad_sch (KiCad schematic)
At the start: 357 parts, among them J1 USB_C_Receptacle_USB2.0, J2 USB_C_Receptacle_USB2.0, SW1 SW_Diode, SW10 SW_Diode, SW100 SW_Diode, SW101 SW_Diode, SW102 SW_Diode, SW103 SW_Diode, SW104 SW_Diode, SW105 SW_Diode, SW106 SW_Diode, SW107 SW_Diode, SW108 SW_Diode, SW109 SW_Diode, SW11 SW_Diode, SW110 SW_Diode, SW111 SW_Diode, SW112 SW_Diode, SW12 SW_Diode, SW13 SW_Diode, SW14 SW_Diode, SW15 SW_Diode, SW16 SW_Diode, SW17 SW_Diode, SW18 SW_Diode, SW19 SW_Diode, SW2 SW_Diode, SW20 SW_Diode, SW21 SW_Diode, SW22 SW_Diode, SW23 SW_Diode, SW24 SW_Diode, SW25 SW_Diode, SW26 SW_Diode, SW27 SW_Diode, SW28 SW_Diode, SW29 SW_Diode, SW3 SW_Diode, SW30 SW_Diode, SW31 SW_Diode, SW32 SW_Diode, SW33 SW_Diode, SW34 SW_Diode, SW35 SW_Diode, SW36 SW_Diode, SW37 SW_Diode, SW38 SW_Diode, SW39 SW_Diode, SW4 SW_Diode, SW40 SW_Diode, SW41 SW_Diode, SW42 SW_Diode, SW43 SW_Diode, SW44 SW_Diode, SW45 SW_Diode, SW46 SW_Diode, SW47 SW_Diode, SW48 SW_Diode, SW49 SW_Diode, SW5 SW_Diode, SW50 SW_Diode, SW51 SW_Diode, SW52 SW_Diode, SW53 SW_Diode, SW54 SW_Diode, SW55 SW_Diode, SW56 SW_Diode, SW57 SW_Diode, SW58 SW_Diode, SW59 SW_Diode, SW6 SW_Diode, SW60 SW_Diode, SW61 SW_Diode, SW62 SW_Diode, SW63 SW_Diode, SW64 SW_Diode, SW65 SW_Diode, SW66 SW_Diode, SW67 SW_Diode, SW68 SW_Diode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

Commit message: add staggered ISO layout
Parts:
- removed C1, C2, C4, C5: C_Small, Capacitor_SMD:C_0603_1608Metric, symbol Device:C_Small
- removed C3, C6: 1µF, Capacitor_SMD:C_0603_1608Metric, symbol Device:C
- removed D103, D109, D110, D111, D112, D15, D16, D17, D18, D19, D20, D37, D38, D39, D40, D41, D55, D58, D59, D60, D61, D62, D77, D78, D79, D94, D95, D96, D97, D98: 1N4148WS, blackwing:D_SOD-323, symbol Diode:1N4148WS
- removed D127, D179, D180, D181, D184, D185, D189, D190, D191, D192, D193, D194, D195, D196, D197, D198, D199, D200, D201, D202, D203, D204, D205, D206, D207, D208, D209, D210, D211: WS2812B-2020, blackwing:LED-WS2812B-2020, symbol ingot:WS2812B-2020
- removed J1, J2: USB_C_Receptacle_USB2.0, Connector_USB:USB_C_Receptacle_GCT_USB4085, symbol Connector:USB_C_Receptacle_USB2.0
- removed JP1: SolderJumper_2_Open, Jumper:SolderJumper-2_P1.3mm_Open_TrianglePad1.0x1.5mm, symbol Jumper:SolderJumper_2_Open
- removed R1, R2, R5, R6: 5.1K, Resistor_SMD:R_0603_1608Metric, symbol Device:R
- removed R3, R4, R7, R8: 22R, Resistor_SMD:R_0603_1608Metric, symbol Device:R
- removed SW109, SW110, SW112, SW15, SW16, SW17, SW18, SW19, SW20, SW37, SW38, SW39, SW40, SW41, SW58, SW59, SW60, SW61, SW77, SW78, SW79, SW94, SW95, SW96, SW97: SW_Diode, blackwing:SW_Cherry_MX_1.00u_PCB, symbol Switch:SW_Push
- removed SW111: SW_Diode, blackwing:SW_Cherry_MX_2.00u_PCB, symbol Switch:SW_Push
- removed SW55: SW_Diode, blackwing:SW_Cherry_MX_1.50u_PCB, symbol Switch:SW_Push
- removed SW62, SW98: SW_Diode, blackwing:SW_Cherry_MX_2.00u_Vertical_PCB, symbol Switch:SW_Push
- removed U1, U2: ATmega32U4-A, Package_QFP:TQFP-44_10x10mm_P0.8mm, symbol MCU_Microchip_ATmega:ATmega32U4-A
- removed Y1, Y2: Crystal, Crystal:Crystal_SMD_HC49-SD_HandSoldering, symbol Device:Crystal
- added D103: 1N4148WS, Diode_SMD:D_SOD-323, symbol Device:D_Small
- added H1: MountingHole, Mounting_Keyboard_Stabilizer:Stabilizer_Cherry_MX_2.00u, symbol Mechanical:MountingHole
- added H2: MountingHole, Mounting_Keyboard_Stabilizer:Stabilizer_Cherry_MX_6.00u, symbol Mechanical:MountingHole
- added U1: RP2040-ZERO, easyeda2kicad:COMM-SMD_RP2040-ZERO, symbol easyeda2kicad:RP2040-ZERO
- D1, D10, D100, D101, D102, D104, D105, D106, D107, D108, D11, D12, D13, D14, D2, D21, D22, D23, D24, D25, D26, D27, D28, D29, D3, D30, D31, D32, D33, D34, D35, D36, D4, D42, D43, D44, D45, D46, D47, D48, D49, D5, D50, D51, D52, D53, D54, D56, D57, D6, D63, D64, D65, D66, D67, D68, D69, D7, D70, D71, D72, D73, D74, D75, D76, D8, D80, D81, D82, D83, D84, D85, D86, D87, D88, D89, D9, D90, D91, D92, D93, D99: footprint blackwing:D_SOD-323 -> Diode_SMD:D_SOD-323; symbol Diode:1N4148WS -> Device:D_Small
- SW102: footprint blackwing:SW_Cherry_MX_6.25u_PCB -> Switch_Keyboard_Cherry_MX:SW_Cherry_MX_PCB_6.00u
- SW105: footprint blackwing:SW_Cherry_MX_1.00u_PCB -> blackwing:SW_Cherry_MX_1.25u_PCB
- SW21, SW4, SW91: footprint blackwing:SW_Cherry_MX_1.50u_PCB -> blackwing:SW_Cherry_MX_1.00u_PCB
- SW34: footprint blackwing:SW_Cherry_MX_1.50u_PCB -> blackwing:SW_Cherry_MX_2.00u_PCB
- SW63: footprint blackwing:SW_Cherry_MX_1.50u_PCB -> blackwing:SW_Cherry_MX_1.75u_PCB
- SW76: footprint blackwing:SW_Cherry_MX_1.50u_PCB -> Switch_Keyboard_Cherry_MX:SW_Cherry_MX_Plate_ISOEnter
- SW80: footprint blackwing:SW_Cherry_MX_1.50u_PCB -> blackwing:SW_Cherry_MX_1.25u_PCB
- SW92: footprint blackwing:SW_Cherry_MX_1.00u_PCB -> blackwing:SW_Cherry_MX_1.75u_PCB
Connections:
- net C09 is gone; now on net C06: SW101.1, SW23.1, SW3.1, SW44.1, SW65.1, SW82.1
- net C10 is gone; now on net C07: SW100.1, SW2.1, SW22.1, SW43.1, SW64.1, SW81.1
- net C11 is gone; now on net C08: SW1.1, SW21.1, SW42.1, SW63.1, SW80.1, SW99.1
- net F-KEY-SDA is gone; now on an unnamed net: D212.3 (SDI)
- net C01: now also SW103.1, SW28.1, SW29.1, SW49.1, SW50.1, SW70.1, SW71.1, SW8.1, SW87.1, SW88.1, SW9.1, U1.12 (GP11); no longer SW10.1, SW104.1, SW105.1, SW11.1, SW31.1, SW32.1, SW52.1, SW53.1, SW73.1, SW74.1, SW90.1, SW91.1
- net C02: now also SW10.1, SW102.2, SW27.1, SW48.1, SW69.1, SW7.1, SW86.1, U1.13 (GP12); no longer SW103.1, SW106.1, SW12.1, SW33.1, SW54.1, SW75.1, SW9.1, SW92.1
- net C03: now also SW104.1, SW11.1, SW26.1, SW31.1, SW47.1, SW52.1, SW6.1, SW68.1, SW73.1, SW85.1, SW90.1, U1.15 (GP14); no longer SW107.1, SW13.1, SW29.1, SW34.1, SW50.1, SW71.1, SW76.1, SW8.1, SW88.1, SW93.1
- net C04: now also SW105.1, SW12.1, SW25.1, SW32.1, SW46.1, SW5.1, SW53.1, SW67.1, SW74.1, SW84.1, SW91.1, U1.16 (GP15); no longer SW108.1, SW14.1, SW28.1, SW35.1, SW49.1, SW56.1, SW7.1, SW70.1, SW87.1
- net C05: now also SW106.1, SW13.1, SW24.1, SW33.1, SW4.1, SW45.1, SW54.1, SW66.1, SW75.1, SW83.1, SW92.1, U1.17 (GP26); no longer SW102.1, SW27.1, SW36.1, SW48.1, SW57.1, SW6.1, SW69.1, SW86.1
- net C06: now also SW107.1, SW14.1, SW34.1, SW76.2, SW93.1, U1.18 (GP27); no longer SW26.1, SW47.1, SW68.1, SW85.1
- net C07: now also SW35.1, SW36.1, SW56.1, SW57.1, U1.5 (GP4); no longer SW25.1, SW46.1, SW5.1, SW67.1, SW84.1
- net C08: now also SW108.1, U1.1 (GP0); no longer SW24.1, SW4.1, SW45.1, SW66.1, SW83.1
- net GND: now also U1.22 (GND); no longer D187.2 (GND)
- net R01: now also U1.20 (GP29); no longer D10.1 (K), D9.1 (K)
- net R02: now also U1.7 (GP6); no longer D29.1 (K), D30.1 (K), D31.1 (K)
- net R03: now also U1.8 (GP7); no longer D50.1 (K), D51.1 (K), D52.1 (K)
- net R04: now also U1.9 (GP8); no longer D71.1 (K), D72.1 (K), D73.1 (K)
- net R05: now also U1.10 (GP9); no longer D88.1 (K), D89.1 (K), D90.1 (K)
- net R06: now also D105.1 (K), D106.1 (K), D103.1 (K), U1.11 (GP10)
- net R07: now also D10.1 (K), D9.1 (K), U1.19 (GP28)
- net R08: now also D29.1 (K), D30.1 (K), D31.1 (K), U1.6 (GP5); no longer D36.1 (K)
- net R09: now also D50.1 (K), D51.1 (K), D52.1 (K), D76.1 (K), U1.4 (GP3); no longer D57.1 (K)
- net R10: now also D36.1 (K), D71.1 (K), D72.1 (K), D73.1 (K), D93.1 (K), U1.3 (GP2); no longer D76.1 (K)
- net R11: now also D107.1 (K), D108.1 (K), D57.1 (K), D88.1 (K), D89.1 (K), D90.1 (K), U1.2 (GP1); no longer D93.1 (K)
- net SDA: now also D188.1 (SDO), U1.14 (GP13); no longer D113.3 (SDI)
- net VBUS: now also U1.23 (5V)
- net at SW103.2: now also D103.2 (A)
- net at D155.1 (SDO): now also D153.1 (SDO); no longer D156.3 (SDI)
- net at D155.3 (SDI): now also D186.3 (SDI); no longer D154.1 (SDO)
- net at D102.2 (A): now also SW102.1; no longer SW102.2
- net at D183.1 (SDO): now also D156.3 (SDI)
- net at D183.3 (SDI): now also D186.1 (SDO); no longer D182.1 (SDO)
- net at D128.3 (SDI): now also D154.1 (SDO)
- net at D76.2 (A): now also SW76.1; no longer SW76.2
- net at D187.3 (SDI): now also D126.1 (SDO); no longer D186.1 (SDO)
- net at D154.3 (SDI): now also D182.1 (SDO); no longer D153.1 (SDO)
- net at D188.3 (SDI): no longer D187.1 (SDO)
- net at D182.3 (SDI): now also D187.1 (SDO)
- net at D224.1 (SDO): now also D113.3 (SDI)
- removed net R12: D105.1 (K), D106.1 (K), D107.1 (K), D108.1 (K)
- no-connect marks 24 -> 2
Other:
- moved on the sheet: D10, D105, D107, D108, D11, D12, D13, D154, D155, D172, D173, D174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

Commit message: design finished
Parts:
- removed H1: MountingHole, Mounting_Keyboard_Stabilizer:Stabilizer_Cherry_MX_2.00u, symbol Mechanical:MountingHole
- removed H2: MountingHole, Mounting_Keyboard_Stabilizer:Stabilizer_Cherry_MX_6.00u, symbol Mechanical:MountingHole
- D1, D10, D100, D101, D102, D103, D104, D105, D106, D107, D108, D11, D12, D13, D14, D2, D21, D22, D23, D24, D25, D26, D27, D28, D29, D3, D30, D31, D32, D33, D34, D35, D36, D4, D42, D43, D44, D45, D46, D47, D48, D49, D5, D50, D51, D52, D53, D54, D56, D57, D6, D63, D64, D65, D66, D67, D68, D69, D7, D70, D71, D72, D73, D74, D75, D76, D8, D80, D81, D82, D83, D84, D85, D86, D87, D88, D89, D9, D90, D91, D92, D93, D99: footprint Diode_SMD:D_SOD-323 -> easyeda2kicad:SOD-323_L1.8-W1.3-LS2.5-RD; symbol Device:D_Small -> easyeda2kicad:1N4148WS-7-F; LCSC Part (none) -> C60580
- D113, D114, D115, D116, D117, D118, D119, D120, D121, D122, D123, D124, D125, D126, D128, D129, D130, D131, D132, D133, D134, D135, D136, D137, D138, D139, D140, D141, D142, D143, D144, D145, D146, D147, D148, D149, D150, D151, D152, D153, D154, D155, D156, D157, D158, D159, D160, D161, D162, D163, D164, D165, D166, D167, D168, D169, D170, D171, D172, D173, D174, D175, D176, D177, D178, D182, D183, D186, D187, D188, D212, D213, D214, D215, D216, D217, D218, D219, D220, D221, D222, D223, D224: footprint blackwing:LED-WS2812B-2020 -> easyeda2kicad:LED-SMD_4P-L2.0-W2.0-BR-1; symbol ingot:WS2812B-2020 -> easyeda2kicad:XL-2020RGBC-WS2812B; LCSC Part (none) -> C5349955
- SW1, SW10, SW100, SW104, SW106, SW107, SW108, SW11, SW12, SW13, SW14, SW2, SW21, SW22, SW23, SW24, SW25, SW26, SW27, SW28, SW29, SW3, SW30, SW31, SW32, SW33, SW35, SW36, SW4, SW43, SW44, SW45, SW46, SW47, SW48, SW49, SW5, SW50, SW51, SW52, SW53, SW54, SW56, SW57, SW6, SW64, SW65, SW66, SW67, SW68, SW69, SW7, SW70, SW71, SW72, SW73, SW74, SW75, SW8, SW81, SW82, SW83, SW84, SW85, SW86, SW87, SW88, SW89, SW9, SW90, SW91, SW93: value SW_Diode -> CPG151101S11-16; footprint blackwing:SW_Cherry_MX_1.00u_PCB -> easyeda2kicad:SMD_KEYBOARD-SW-1.00; symbol Switch:SW_Push -> easyeda2kicad:CPG151101S11-16_C41430893; LCSC Part (none) -> C41430893
- SW101, SW103, SW105, SW80, SW99: value SW_Diode -> CPG151101S11-16; footprint blackwing:SW_Cherry_MX_1.25u_PCB -> easyeda2kicad:SMD_KEYBOARD-SW-1.25; symbol Switch:SW_Push -> easyeda2kicad:CPG151101S11-16_C41430893; LCSC Part (none) -> C41430893
- SW102: value SW_Diode -> CPG151101S11-16; footprint Switch_Keyboard_Cherry_MX:SW_Cherry_MX_PCB_6.00u -> easyeda2kicad:SMD_KEYBOARD-SW-6.00; symbol Switch:SW_Push -> easyeda2kicad:CPG151101S11-16_C41430893; LCSC Part (none) -> C41430893
- SW34: value SW_Diode -> CPG151101S11-16; footprint blackwing:SW_Cherry_MX_2.00u_PCB -> easyeda2kicad:SMD_KEYBOARD-SW-2.00; symbol Switch:SW_Push -> easyeda2kicad:CPG151101S11-16_C41430893; LCSC Part (none) -> C41430893
- SW42: value SW_Diode -> CPG151101S11-16; footprint blackwing:SW_Cherry_MX_1.50u_PCB -> easyeda2kicad:SMD_KEYBOARD-SW-1.50; symbol Switch:SW_Push -> easyeda2kicad:CPG151101S11-16_C41430893; LCSC Part (none) -> C41430893
- SW63, SW92: value SW_Diode -> CPG151101S11-16; footprint blackwing:SW_Cherry_MX_1.75u_PCB -> easyeda2kicad:SMD_KEYBOARD-SW-1.75; symbol Switch:SW_Push -> easyeda2kicad:CPG151101S11-16_C41430893; LCSC Part (none) -> C41430893
- SW76: value SW_Diode -> CPG151101S11-16; footprint Switch_Keyboard_Cherry_MX:SW_Cherry_MX_Plate_ISOEnter -> easyeda2kicad:SMD_KEYBOARD-SW-ENTER-ISO; symbol Switch:SW_Push -> easyeda2kicad:CPG151101S11-16_C41430893; LCSC Part (none) -> C41430893
Connections:
- net C02: now also SW102.1; no longer SW102.2
- net C06: now also SW76.1; no longer SW76.2
- net GND: now also D187.2 (GND)
- net SDA: now also D188.3 (DI); no longer D188.1 (SDO)
- net at D155.1 (DO): now also D186.3 (DI); no longer D153.1 (SDO)
- net at D155.3 (DI): now also D153.1 (DO); no longer D186.3 (SDI)
- net at D102.2 (A): now also SW102.2; no longer SW102.1
- net at D212.3 (DI): now also D188.1 (DO); no longer D188.3 (SDI)
- net at D76.2 (A): now also SW76.2; no longer SW76.1
