File: plate/pcb.kicad_pcb (KiCad board)
At the start: 2 copper layers, 323 x 133 mm, 83 parts, among them SW1 SW_Diode, SW10 SW_Diode, SW100 SW_Diode, SW101 SW_Diode, SW102 SW_Diode, SW103 SW_Diode, SW104 SW_Diode, SW105 SW_Diode, SW106 SW_Diode, SW107 SW_Diode, SW108 SW_Diode, SW11 SW_Diode, SW12 SW_Diode, SW13 SW_Diode, SW14 SW_Diode, SW2 SW_Diode, SW21 SW_Diode, SW22 SW_Diode, SW23 SW_Diode, SW24 SW_Diode, SW25 SW_Diode, SW26 SW_Diode, SW27 SW_Diode, SW28 SW_Diode, SW29 SW_Diode, SW3 SW_Diode, SW30 SW_Diode, SW31 SW_Diode, SW32 SW_Diode, SW33 SW_Diode, SW34 SW_Diode, SW35 SW_Diode, SW36 SW_Diode, SW4 SW_Diode, SW42 SW_Diode, SW43 SW_Diode, SW44 SW_Diode, SW45 SW_Diode, SW46 SW_Diode, SW47 SW_Diode, SW48 SW_Diode, SW49 SW_Diode, SW5 SW_Diode, SW50 SW_Diode, SW51 SW_Diode, SW52 SW_Diode, SW53 SW_Diode, SW54 SW_Diode, SW56 SW_Diode, SW57 SW_Diode, SW6 SW_Diode, SW63 SW_Diode, SW64 SW_Diode, SW65 SW_Diode, SW66 SW_Diode, SW67 SW_Diode, SW68 SW_Diode, SW69 SW_Diode, SW7 SW_Diode, SW70 SW_Diode, SW71 SW_Diode, SW72 SW_Diode, SW73 SW_Diode, SW74 SW_Diode, SW75 SW_Diode, SW76 SW_Diode, SW8 SW_Diode, SW80 SW_Diode, SW81 SW_Diode, SW82 SW_Diode, SW83 SW_Diode, SW84 SW_Diode, SW85 SW_Diode, SW86 SW_Diode, SW87 SW_Diode, SW88 SW_Diode, SW89 SW_Diode, SW9 SW_Diode, SW90 SW_Diode, SW91 SW_Diode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

Commit message: drc clean
Parts:
- added H1: MountingHole_Pad, blackwing:dummy_via, F.Cu at (131.0, 92.1)
Routing:
- net (no net): vias 1 -> 0
- added copper zone on B.Cu, net GND
- added copper zone on F.Cu, net GND
- removed copper zone on B.Cu, net (none)
- removed copper zone on F.Cu, net (none)
Changed lines of the file:
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@@
 		(pad_to_mask_clearance 0)
 		(allow_soldermask_bridges_in_footprints no)
-		(grid_origin 282.46 -23.42)
+		(grid_origin 249.21 -18.67)
 		(pcbplotparams
 			(layerselection 0x00010fc_ffffffff)
@@
 	)
 	(net 0 "")
+	(net 1 "GND")
 	(footprint "blackwing:CUTOUT_CHERRY_MX_1.00u"
 		(layer "F.Cu")
@@
 		)
 		(fp_rect
-			(start -62.04 -4.42)
-			(end 57.0225 14.63)
+			(start -59.54 -4.42)
+			(end 54.46 14.58)
 			(stroke
 				(width 0.1)
@@
 		)
 	)
+	(footprint "blackwing:dummy_via"
+		(layer "F.Cu")
+		(at 130.96 92.08)
+		(descr "Circular Fiducial, 0.5mm bare copper, 1mm soldermask opening (Level C)")
+		(tags "fiducial")
+		(property "Reference" "H1"
+			(at 0 -1.5 0)
+			(layer "F.SilkS")
+			(hide yes)
+			(effects
+				(font
+					(size 1 1)
+					(thickness 0.15)
+				)
+			)
+		)
+		(property "Value" "MountingHole_Pad"
+			(at 0 1.5 0)
+			(layer "F.Fab")
+			(effects
+				(font
+					(size 1 1)
+					(thickness 0.15)
+				)
+			)
+		)
+		(property "Footprint" "blackwing:dummy_via"
+			(at 0 0 0)
+			(unlocked yes)
+			(layer "F.Fab")
+			(hide yes)
+			(effects
+				(font
+					(size 1.27 1.27)
+					(thickness 0.15)
+				)
+			)
+		)
+		(property "Datasheet" ""
+			(at 0 0 0)
+			(unlocked yes)
+			(layer "F.Fab")
+			(hide yes)
+			(effects
+				(font
+					(size 1.27 1.27)
+					(thickness 0.15)
+				)
+			)
+		)
+		(property "Description" "Mounting Hole with connection"
+			(at 0 0 0)
+			(unlocked yes)
+			(layer "F.Fab")
+			(hide yes)
+			(effects
+				(font
+					(size 1.27 1.27)
+					(thickness 0.15)
+				)
+			)
+		)
+		(property ki_fp_filters "MountingHole*Pad*")
+		(sheetname "Root")
+		(sheetfile "pcb.kicad_sch")
+		(attr smd exclude_from_bom)
+		(fp_circle
+			(center 0 0)
+			(end 0.75 0)
+			(stroke
+				(width 0.05)
+				(type solid)
+			)
+			(fill none)
+			(layer "F.CrtYd")
+		)
+		(fp_circle
+			(center 0 0)
+			(end 0.5 0)
+			(stroke
+				(width 0.1)
+				(type solid)
+			)
+			(fill none)
+			(layer "F.Fab")
+		)
+		(fp_text user "${REFERENCE}"
+			(at 0 0 0)
+			(layer "F.Fab")
+			(effects
+				(font
+					(size 0.2 0.2)
+					(thickness 0.04)
+				)
+			)
+		)
+		(pad "1" thru_hole circle
+			(at 0 0)
+			(size 0.8 0.8)
+			(drill 0.4)
+			(layers "*.Cu" "*.Mask")
+			(remove_unused_layers no)
+			(net 1 "GND")
+			(pinfunction "1")
+			(pintype "input")
+			(solder_mask_margin 0.25)
+			(clearance 0.25)
+			(zone_connect 2)
+		)
+	)
 	(footprint "blackwing:CUTOUT_CHERRY_MX_1.00u"
 		(layer "F.Cu")
@@
 		(layer "Edge.Cuts")
 	)
-	(via
-		(at 130.96 92.08)
-		(size 0.8)
-		(drill 0.4)
-		(layers "F.Cu" "B.Cu")
-		(net 0)
-	)
 	(zone
-		(net 0)
-		(net_name "")
+		(net 1)
+		(net_name "GND")
 		(layers "F&B.Cu")
 		(hatch edge 0.508)
