File: plate/pcb.kicad_sch (KiCad schematic)
At the start: 83 parts, among them SW1 SW_Diode, SW10 SW_Diode, SW100 SW_Diode, SW101 SW_Diode, SW102 SW_Diode, SW103 SW_Diode, SW104 SW_Diode, SW105 SW_Diode, SW106 SW_Diode, SW107 SW_Diode, SW108 SW_Diode, SW11 SW_Diode, SW12 SW_Diode, SW13 SW_Diode, SW14 SW_Diode, SW2 SW_Diode, SW21 SW_Diode, SW22 SW_Diode, SW23 SW_Diode, SW24 SW_Diode, SW25 SW_Diode, SW26 SW_Diode, SW27 SW_Diode, SW28 SW_Diode, SW29 SW_Diode, SW3 SW_Diode, SW30 SW_Diode, SW31 SW_Diode, SW32 SW_Diode, SW33 SW_Diode, SW34 SW_Diode, SW35 SW_Diode, SW36 SW_Diode, SW4 SW_Diode, SW42 SW_Diode, SW43 SW_Diode, SW44 SW_Diode, SW45 SW_Diode, SW46 SW_Diode, SW47 SW_Diode, SW48 SW_Diode, SW49 SW_Diode, SW5 SW_Diode, SW50 SW_Diode, SW51 SW_Diode, SW52 SW_Diode, SW53 SW_Diode, SW54 SW_Diode, SW56 SW_Diode, SW57 SW_Diode, SW6 SW_Diode, SW63 SW_Diode, SW64 SW_Diode, SW65 SW_Diode, SW66 SW_Diode, SW67 SW_Diode, SW68 SW_Diode, SW69 SW_Diode, SW7 SW_Diode, SW70 SW_Diode, SW71 SW_Diode, SW72 SW_Diode, SW73 SW_Diode, SW74 SW_Diode, SW75 SW_Diode, SW76 SW_Diode, SW8 SW_Diode, SW80 SW_Diode, SW81 SW_Diode, SW82 SW_Diode, SW83 SW_Diode, SW84 SW_Diode, SW85 SW_Diode, SW86 SW_Diode, SW87 SW_Diode, SW88 SW_Diode, SW89 SW_Diode, SW9 SW_Diode, SW90 SW_Diode, SW91 SW_Diode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

Commit message: drc clean
Parts:
- added H1: MountingHole_Pad, blackwing:dummy_via, symbol Mechanical:MountingHole_Pad
- SW1, SW10, SW100, SW101, SW102, SW103, SW104, SW105, SW106, SW107, SW108, SW11, SW12, SW13, SW14, SW2, SW21, SW22, SW23, SW24, SW25, SW26, SW27, SW28, SW29, SW3, SW30, SW31, SW32, SW33, SW34, SW35, SW36, SW4, SW42, SW43, SW44, SW45, SW46, SW47, SW48, SW49, SW5, SW50, SW51, SW52, SW53, SW54, SW56, SW57, SW6, SW63, SW64, SW65, SW66, SW67, SW68, SW69, SW7, SW70, SW71, SW72, SW73, SW74, SW75, SW76, SW8, SW80, SW81, SW82, SW83, SW84, SW85, SW86, SW87, SW88, SW89, SW9, SW90, SW91, SW92, SW93, SW99: symbol easyeda2kicad:CPG151101S11-16_C41430893 -> easyeda2kicad:SW_CUTOUT
Connections:
- new net GND: H1.1
